File: main_pcb/IRIS-OHYAMA-IHK-T35-I2C-Controller.sch (KiCad schematic (older format))
At the start: 52 parts, among them CN1 Conn_01x05, J1 Grove, J2 Conn_01x06, J3 thermistor, Q1 Q_NMOS_DGS, Q2 Q_NMOS_DGS, Q3 Q_NMOS_DGS, Q4 Q_NMOS_DGS, U1 74HC164, U2 ATmega328P-MU

Commit message: Change mosfet to GSD
Parts:
- Q1, Q2, Q3, Q4: value Q_NMOS_DGS -> Q_NMOS_GSD; symbol Device:Q_NMOS_DGS -> Device:Q_NMOS_GSD
Changed lines of the file:
@@
 PIN_POWER_OIL
 $Comp
-L Device:Q_NMOS_DGS Q2
+L Device:Q_NMOS_GSD Q2
 U 1 1 5E7B71FA
 P 2250 6600
 F 0 "Q2" H 2454 6646 50  0000 L CNN
-F 1 "Q_NMOS_DGS" H 2454 6555 50  0000 L CNN
+F 1 "Q_NMOS_GSD" H 2454 6555 50  0000 L CNN
 F 2 "Package_TO_SOT_SMD:SOT-23" H 2450 6700 50  0001 C CNN
 F 3 "~" H 2250 6600 50  0001 C CNN
@@
 PIN_POWER_DOWN
 $Comp
-L Device:Q_NMOS_DGS Q4
+L Device:Q_NMOS_GSD Q4
 U 1 1 5E7CD8E8
 P 4000 6650
 F 0 "Q4" H 4204 6696 50  0000 L CNN
-F 1 "Q_NMOS_DGS" H 4204 6605 50  0000 L CNN
+F 1 "Q_NMOS_GSD" H 4204 6605 50  0000 L CNN
 F 2 "Package_TO_SOT_SMD:SOT-23" H 4200 6750 50  0001 C CNN
 F 3 "~" H 4000 6650 50  0001 C CNN
@@
 PIN_POWER_NORMAL
 $Comp
-L Device:Q_NMOS_DGS Q1
+L Device:Q_NMOS_GSD Q1
 U 1 1 5E7CF502
 P 2250 5400
 F 0 "Q1" H 2454 5446 50  0000 L CNN
-F 1 "Q_NMOS_DGS" H 2454 5355 50  0000 L CNN
+F 1 "Q_NMOS_GSD" H 2454 5355 50  0000 L CNN
 F 2 "Package_TO_SOT_SMD:SOT-23" H 2450 5500 50  0001 C CNN
 F 3 "~" H 2250 5400 50  0001 C CNN
@@
 PIN_POWER_UP
 $Comp
-L Device:Q_NMOS_DGS Q3
+L Device:Q_NMOS_GSD Q3
 U 1 1 5E7D1335
 P 4000 5450
 F 0 "Q3" H 4204 5496 50  0000 L CNN
-F 1 "Q_NMOS_DGS" H 4204 5405 50  0000 L CNN
+F 1 "Q_NMOS_GSD" H 4204 5405 50  0000 L CNN
 F 2 "Package_TO_SOT_SMD:SOT-23" H 4200 5550 50  0001 C CNN
 F 3 "~" H 4000 5450 50  0001 C CNN
